File: LoadSwitch.kicad_pcb (KiCad board)
At the start: 2 copper layers, 36.6 x 26.9 mm, 21 parts, among them IC1 LTC4359, P1 CONN_01X03, P2 CONN_01X03, P3 CONN_01X02, P4 CONN_01X02, Q1 FDMS86101, Q2 FDMS86101, U1 LTV-817

Commit message: Gerber erstellt
Other:
- rule pad_to_mask_clearance: 0 -> 0.1
Changed lines of the file:
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@@
     (pad_size 1.89 1.57)
     (pad_drill 0)
-    (pad_to_mask_clearance 0)
+    (pad_to_mask_clearance 0.1)
     (aux_axis_origin 0 0)
     (visible_elements FFFFF77F)
     (pcbplotparams
-      (layerselection 0x00030_80000001)
-      (usegerberextensions false)
+      (layerselection 0x010f0_80000001)
+      (usegerberextensions true)
       (excludeedgelayer true)
       (linewidth 0.100000)
@@
       (psa4output false)
       (plotreference true)
-      (plotvalue true)
+      (plotvalue false)
       (plotinvisibletext false)
       (padsonsilk false)
@@
       (outputformat 1)
       (mirror false)
-      (drillshape 1)
+      (drillshape 0)
       (scaleselection 1)
-      (outputdirectory ""))
+      (outputdirectory switch-gerber/))
   )
   (net 0 "")
